File: RaspberryPi-breakout.brd (EAGLE design)
At the start: 21.9 x 35.2 mm, 3 parts

Commit message: Pass #1
Other:
- outline, holes or cut-outs redrawn
- board text added: "3V3"
- board text added: "5V"
- board text removed: "+3V3"
- board text removed: "+5V"
Changed lines of the file:
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@@
 <setting verticaltext="up"/>
 </settings>
-<grid distance="0.3175" unitdist="mm" unit="mm" style="lines" multiple="1" display="no" altdistance="0.025" altunitdist="inch" altunit="inch"/>
+<grid distance="0.75" unitdist="mil" unit="mil" style="lines" multiple="1" display="yes" altdistance="0.025" altunitdist="inch" altunit="inch"/>
 <layers>
 <layer number="1" name="Top" color="4" fill="1" visible="yes" active="yes"/>
@@
 <board>
 <plain>
-<wire x1="0" y1="0" x2="21.895" y2="0" width="0" layer="20"/>
 <wire x1="21.895" y1="0" x2="21.895" y2="35.2325" width="0" layer="20"/>
 <wire x1="21.895" y1="35.2325" x2="0" y2="35.2325" width="0" layer="20"/>
-<wire x1="0" y1="35.2325" x2="0" y2="0" width="0" layer="20"/>
-<text x="14.2875" y="31.75" size="0.8128" layer="21">+5V</text>
-<text x="14.2875" y="29.21" size="0.8128" layer="21">+5V</text>
-<text x="14.2875" y="26.67" size="0.8128" layer="21">GND</text>
-<text x="14.2875" y="16.51" size="0.8128" layer="21">GND</text>
-<text x="14.2875" y="8.89" size="0.8128" layer="21">GND</text>
-<text x="6.35" y="1.27" size="0.8128" layer="21">GND</text>
-<text x="6.35" y="21.59" size="0.8128" layer="21">GND</text>
+<text x="15.24" y="31.4325" size="0.8128" layer="21" rot="R90">5V</text>
+<text x="7.62" y="2.54" size="0.8128" layer="21" rot="SR270">GND</text>
 <text x="14.2875" y="13.97" size="0.6096" layer="21">GPIO23</text>
 <text x="14.2875" y="11.43" size="0.6096" layer="21">GPIO24</text>
@@
 <text x="5.715" y="6.985" size="0.6096" layer="21">GPIO9</text>
 <text x="5.715" y="9.525" size="0.6096" layer="21">GPIO10</text>
-<text x="5.715" y="11.43" size="0.8128" layer="21">+3V3</text>
-<text x="5.715" y="31.75" size="0.8128" layer="21">+3V3</text>
 <text x="5.715" y="14.2875" size="0.6096" layer="21">GPIO22</text>
 <text x="5.715" y="16.8275" size="0.6096" layer="21">GPIO21</text>
@@
 <text x="14.2875" y="20.955" size="0.8128" layer="21">RX</text>
 <text x="14.2875" y="23.495" size="0.8128" layer="21">TX</text>
+<text x="15.24" y="28.8925" size="0.8128" layer="21" rot="R90">5V</text>
+<text x="7.62" y="12.7" size="0.8128" layer="21" rot="SR270">3V3</text>
+<text x="7.62" y="22.86" size="0.8128" layer="21" rot="SR270">GND</text>
+<text x="15.24" y="25.7175" size="0.8128" layer="21" rot="R90">GND</text>
+<text x="15.24" y="15.875" size="0.8128" layer="21" rot="R90">GND</text>
+<text x="15.24" y="7.9375" size="0.8128" layer="21" rot="R90">GND</text>
+<wire x1="-0.0506" y1="0" x2="-0.0506" y2="35.2325" width="0" layer="20"/>
+<wire x1="21.8569" y1="0.00905" x2="-0.0381" y2="0.00905" width="0" layer="20"/>
+<text x="7.7343" y="32.9692" size="0.8128" layer="21" rot="SR270">3V3</text>
 </plain>
 <attributes>
